File: hardware/imu.kicad_sch (KiCad schematic)
At the start: 3 parts, among them U14 LSM6DSV16XTR

Commit message: Standardize repo: .gitignore, README, license, remove orphaned files
- Standardize .gitignore to match ecosystem template
- Fix README: correct GitHub URL, remove generic sections, remove nonexistent dirs
- Replace LICENSE stub with full CERN-OHL-S-2.0 text
- Remove orphaned schematics (baro, blackbox, compass, elrs, leds) — not in ECO variant
- Delete self-referential symlink and parent OpenFC production leftovers
- Add new footprints and 3D models (SIM, TF connectors)

Co-Authored-By: Claude Opus 4.6 (1M context) <noreply@anthropic.com>
Connections:
- net SPI0.CLKIN: now reaches U14.9 (INT2)
- no-connect marks 3 -> 2

Commit message: WIP: schematic updates, library modernization, audit tooling
Schematic changes (user):
- Add ADC bypass caps on CURRENT/RSSI/EXTERNAL (1k + 100nF RC filter)
- Add IMU GYRO_CS 10k pull-up to +3.3V
- Reverse P1 ESC 8-pin JST SH pinout to BF standard
  (pin1=V+, pin2=GND, pin3=Current, pin5-8=M1-M4)
- SD card (blackbox) sub-sheet with SPI1 + FLASH_CS + decoupling
- Other sub-sheet cleanup (rp2350a, osd, pads, power, imu)

Footprint library:
- Convert all 62 legacy (module ...) footprints to modern
  (footprint ...) format via pcbnew API — fixes kicad-sch-api
  "footprint not found" errors

Tooling:
- Add hardware/tools/audit_design.py (BF-rule design audit script)
- Add hardware/tools/design_audit.md (audit report output)

Docs:
- Update CLAUDE.md: current GPIO map, corrected power tree net names,
  open issues list (CRIT-2..5), connector verification status

Co-Authored-By: Claude Opus 4.6 (1M context) <noreply@anthropic.com>
Parts:
- renumbered C41 to C35, C34 to C36, U14 to U9
Changed lines of the file:
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@@
 		(dnp no)
 		(fields_autoplaced yes)
-		(property "Reference" "#PWR05"
+		(property "Reference" "#PWR0130"
 			(at 83.82 46.99 0)
 			(hide yes)
@@
 			(project "OpenFC"
 				(path "/fb88b6f9-ee39-4640-a9d4-04a17ceeac64/757ed1e6-9a5f-4a0e-a946-254eae8dfb0d"
-					(reference "#PWR05")
+					(reference "#PWR0130")
 					(unit 1)
 				)
@@
 		(dnp no)
 		(fields_autoplaced yes)
-		(property "Reference" "#PWR031"
+		(property "Reference" "#PWR0125"
 			(at 45.72 99.06 0)
 			(hide yes)
@@
 			(project "OpenFC"
 				(path "/fb88b6f9-ee39-4640-a9d4-04a17ceeac64/757ed1e6-9a5f-4a0e-a946-254eae8dfb0d"
-					(reference "#PWR031")
+					(reference "#PWR0125")
 					(unit 1)
 				)
@@
 		(dnp no)
 		(fields_autoplaced yes)
-		(property "Reference" "#PWR010"
+		(property "Reference" "#PWR0131"
 			(at 83.82 57.15 0)
 			(hide yes)
@@
 			(project "OpenFC"
 				(path "/fb88b6f9-ee39-4640-a9d4-04a17ceeac64/757ed1e6-9a5f-4a0e-a946-254eae8dfb0d"
-					(reference "#PWR010")
+					(reference "#PWR0131")
 					(unit 1)
 				)
@@
 		(in_pos_files yes)
 		(dnp no)
-		(property "Reference" "C41"
+		(property "Reference" "C35"
 			(at 62.23 44.45 0)
 			(show_name no)
@@
 			(project "OpenFC"
 				(path "/fb88b6f9-ee39-4640-a9d4-04a17ceeac64/757ed1e6-9a5f-4a0e-a946-254eae8dfb0d"
-					(reference "C41")
+					(reference "C35")
 					(unit 1)
 				)
@@
 		(dnp no)
 		(fields_autoplaced yes)
-		(property "Reference" "#PWR0144"
+		(property "Reference" "#PWR0127"
 			(at 71.12 43.18 0)
 			(hide yes)
@@
 			(project "OpenFC"
 				(path "/fb88b6f9-ee39-4640-a9d4-04a17ceeac64/757ed1e6-9a5f-4a0e-a946-254eae8dfb0d"
-					(reference "#PWR0144")
+					(reference "#PWR0127")
 					(unit 1)
 				)
@@
 		(in_pos_files yes)
 		(dnp no)
-		(property "Reference" "U14"
+		(property "Reference" "U9"
 			(at 60.96 68.326 0)
 			(show_name no)
@@
 			(project "OpenFC"
 				(path "/fb88b6f9-ee39-4640-a9d4-04a17ceeac64/757ed1e6-9a5f-4a0e-a946-254eae8dfb0d"
-					(reference "U14")
+					(reference "U9")
 					(unit 1)
 				)
@@
 		(dnp no)
 		(fields_autoplaced yes)
-		(property "Reference" "#PWR0146"
+		(property "Reference" "#PWR0126"
 			(at 62.23 57.15 0)
 			(hide yes)
@@
 			(project "OpenFC"
 				(path "/fb88b6f9-ee39-4640-a9d4-04a17ceeac64/757ed1e6-9a5f-4a0e-a946-254eae8dfb0d"
-					(reference "#PWR0146")
+					(reference "#PWR0126")
 					(unit 1)
 				)
@@
 		(dnp no)
 		(fields_autoplaced yes)
-		(property "Reference" "#PWR0145"
+		(property "Reference" "#PWR0128"
 			(at 72.39 99.06 0)
 			(hide yes)
@@
 			(project "OpenFC"
 				(path "/fb88b6f9-ee39-4640-a9d4-04a17ceeac64/757ed1e6-9a5f-4a0e-a946-254eae8dfb0d"
-					(reference "#PWR0145")
+					(reference "#PWR0128")
 					(unit 1)
 				)
@@
 		(in_pos_files yes)
 		(dnp no)
-		(property "Reference" "C34"
+		(property "Reference" "C36"
 			(at 83.82 44.45 0)
 			(show_name no)
@@
 			(project "OpenFC"
 				(path "/fb88b6f9-ee39-4640-a9d4-04a17ceeac64/757ed1e6-9a5f-4a0e-a946-254eae8dfb0d"
-					(reference "C34")
+					(reference "C36")
 					(unit 1)
 				)
@@
 		(dnp no)
 		(fields_autoplaced yes)
-		(property "Reference" "#PWR078"
+		(property "Reference" "#PWR0129"
 			(at 73.66 60.96 0)
 			(hide yes)
@@
 			(project "OpenFC"
 				(path "/fb88b6f9-ee39-4640-a9d4-04a17ceeac64/757ed1e6-9a5f-4a0e-a946-254eae8dfb0d"
-					(reference "#PWR078")
-					(unit 1)
-				)
+					(reference "#PWR0129")
+					(unit 1)
+				)
