File: hardware/osd.kicad_sch (KiCad schematic)
At the start: 17 parts, among them U34 TLV3201AIDBVR, U35 SN74LVC1G3157DTBR, U38 TLV9061IDPWR

Commit message: WIP: schematic updates, library modernization, audit tooling
Schematic changes (user):
- Add ADC bypass caps on CURRENT/RSSI/EXTERNAL (1k + 100nF RC filter)
- Add IMU GYRO_CS 10k pull-up to +3.3V
- Reverse P1 ESC 8-pin JST SH pinout to BF standard
  (pin1=V+, pin2=GND, pin3=Current, pin5-8=M1-M4)
- SD card (blackbox) sub-sheet with SPI1 + FLASH_CS + decoupling
- Other sub-sheet cleanup (rp2350a, osd, pads, power, imu)

Footprint library:
- Convert all 62 legacy (module ...) footprints to modern
  (footprint ...) format via pcbnew API — fixes kicad-sch-api
  "footprint not found" errors

Tooling:
- Add hardware/tools/audit_design.py (BF-rule design audit script)
- Add hardware/tools/design_audit.md (audit report output)

Docs:
- Update CLAUDE.md: current GPIO map, corrected power tree net names,
  open issues list (CRIT-2..5), connector verification status

Co-Authored-By: Claude Opus 4.6 (1M context) <noreply@anthropic.com>
Parts:
- renumbered C64 to C38, C49 to C39, C66 to C40, C69 to C41, C3 to C42, R21 to R41, R30 to R42, R46 to R43, R45 to R44, R27 to R45, R48 to R46, R49 to R47, R47 to R48, U35 to U18, U38 to U19, U34 to U20

Commit message: V0.3 routed: pin remap, footprint fixes, EMC checklist, DFM prep
Schematic (user):
- OSD pins remapped to GPIO4-6 (OSD_W/OSD_EN/OSD_SYNC consecutive
  for FB_OSD PIO driver per BF PR#14882)
- SBUS inverter stays on GPIO9 (valid UART1_RX)
- Beeper moved to GPIO36
- Various sub-sheet updates

PCB:
- Full board routed, bottom-side component placement
- Resistor footprints: C_0201 -> R_0201 for correct 3D models
- Capacitor 3D model paths fixed (were pointing to R_0201)
- SD card footprint 3D path fixed (${KIPRJMOD}/lib.3dshapes/)
- 2 footprint 3D paths fixed (SIM, TF-01A: /lib.3dshapes -> ${KIPRJMOD})

Tooling & docs:
- Add EMC checklist (hardware/tools/EMC_CHECKLIST.md)
- Add EMC note script (hardware/tools/add_emc_note.py)
- Update CLAUDE.md: LMR51430 drop-in upgrade noted, connector
  verification, OSD pin mapping

Co-Authored-By: Claude Opus 4.6 (1M context) <noreply@anthropic.com>
Parts:
- R41, R42, R43, R44, R45, R46, R47, R48: footprint Capacitor_SMD:C_0201_0603Metric -> Resistor_SMD:R_0201_0603Metric
Changed lines of the file:
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@@
 			)
 		)
-		(property "Footprint" "Capacitor_SMD:C_0201_0603Metric"
+		(property "Footprint" "Resistor_SMD:R_0201_0603Metric"
 			(at 97.79 169.418 90)
 			(hide yes)
@@
 			)
 		)
-		(property "Footprint" "Capacitor_SMD:C_0201_0603Metric"
+		(property "Footprint" "Resistor_SMD:R_0201_0603Metric"
 			(at 179.578 186.69 90)
 			(hide yes)
@@
 			)
 		)
-		(property "Footprint" "Capacitor_SMD:C_0201_0603Metric"
+		(property "Footprint" "Resistor_SMD:R_0201_0603Metric"
 			(at 110.998 161.29 90)
 			(hide yes)
@@
 			)
 		)
-		(property "Footprint" "Capacitor_SMD:C_0201_0603Metric"
+		(property "Footprint" "Resistor_SMD:R_0201_0603Metric"
 			(at 210.82 166.878 90)
 			(hide yes)
@@
 			)
 		)
-		(property "Footprint" "Capacitor_SMD:C_0201_0603Metric"
+		(property "Footprint" "Resistor_SMD:R_0201_0603Metric"
 			(at 110.998 173.99 90)
 			(hide yes)
@@
 			)
 		)
-		(property "Footprint" "Capacitor_SMD:C_0201_0603Metric"
+		(property "Footprint" "Resistor_SMD:R_0201_0603Metric"
 			(at 96.012 115.57 90)
 			(hide yes)
@@
 			)
 		)
-		(property "Footprint" "Capacitor_SMD:C_0201_0603Metric"
+		(property "Footprint" "Resistor_SMD:R_0201_0603Metric"
 			(at 129.54 107.442 90)
 			(hide yes)
@@
 			)
 		)
-		(property "Footprint" "Capacitor_SMD:C_0201_0603Metric"
+		(property "Footprint" "Resistor_SMD:R_0201_0603Metric"
 			(at 199.39 182.118 90)
 			(hide yes)
