File: hardware/pads.kicad_sch (KiCad schematic)
At the start: 56 parts, among them J1 5V, J13 5V, J14 5V, J15 5V, J16 5V, J17 5V, J18 5V, J19 5V, J2 5V, J20 5V, J21 5V, J22 5V, J23 5V, J24 5V, J25 5V, J27 5V, J28 5V, J29 5V, J3 5V, J30 5V, J32 5V, J33 5V, J34 5V, J35 5V, J36 5V, J37 5V, J38 5V, J39 5V, J4 5V, J40 5V, J41 5V, J42 5V, J43 5V, J44 5V, J45 5V, J46 5V, J47 5V, J48 5V, J49 5V, J5 5V, J50 5V, J51 5V, J52 5V, J53 5V, J54 5V, J55 5V, J56 5V, J57 5V, J58 5V, J59 5V, J6 5V, J7 5V, J8 5V, J9 5V, P1 SM08B-SRSS-TB(LF)(SN), U1 SM06B-SRSS-TB(LF)(SN)

Commit message: Standardize repo: .gitignore, README, license, remove orphaned files
- Standardize .gitignore to match ecosystem template
- Fix README: correct GitHub URL, remove generic sections, remove nonexistent dirs
- Replace LICENSE stub with full CERN-OHL-S-2.0 text
- Remove orphaned schematics (baro, blackbox, compass, elrs, leds) — not in ECO variant
- Delete self-referential symlink and parent OpenFC production leftovers
- Add new footprints and 3D models (SIM, TF connectors)

Co-Authored-By: Claude Opus 4.6 (1M context) <noreply@anthropic.com>
Parts:
- J1, J16, J17, J18, J19, J2, J20, J21, J22, J23, J24, J25, J27, J28, J29, J3, J30, J32, J33, J34, J35, J36, J37, J38, J39, J4, J40, J43, J44, J45, J46, J49, J5, J50, J51, J52, J53, J54, J55, J56, J57, J58, J59, J6, J7, J8, J9: now left out of the parts list
- J13, J14, J15, J41, J42, J47, J48: now fitted; now left out of the parts list
Connections:
- net +BATT: now also J27.1 (Pin_1)

Commit message: WIP: schematic updates, library modernization, audit tooling
Schematic changes (user):
- Add ADC bypass caps on CURRENT/RSSI/EXTERNAL (1k + 100nF RC filter)
- Add IMU GYRO_CS 10k pull-up to +3.3V
- Reverse P1 ESC 8-pin JST SH pinout to BF standard
  (pin1=V+, pin2=GND, pin3=Current, pin5-8=M1-M4)
- SD card (blackbox) sub-sheet with SPI1 + FLASH_CS + decoupling
- Other sub-sheet cleanup (rp2350a, osd, pads, power, imu)

Footprint library:
- Convert all 62 legacy (module ...) footprints to modern
  (footprint ...) format via pcbnew API — fixes kicad-sch-api
  "footprint not found" errors

Tooling:
- Add hardware/tools/audit_design.py (BF-rule design audit script)
- Add hardware/tools/design_audit.md (audit report output)

Docs:
- Update CLAUDE.md: current GPIO map, corrected power tree net names,
  open issues list (CRIT-2..5), connector verification status

Co-Authored-By: Claude Opus 4.6 (1M context) <noreply@anthropic.com>
Parts:
- renumbered J9 to J1, J21 to J10, J52 to J11, J43 to J12, J51 to J13, J42 to J14, J8 to J15, J22 to J17, J7 to J18, J17 to J19, J56 to J2, J23 to J20, J40 to J21, J6 to J22, J18 to J23, J30 to J24, J39 to J25, J5 to J26, J50 to J27, J59 to J28, J27 to J29, J13 to J3, J49 to J30, J25 to J31, J24 to J33, J33 to J34, J4 to J35, J41 to J36, J3 to J37, J58 to J38, J2 to J39, J19 to J4, J48 to J40, J1 to J41, J47 to J42, J46 to J43, J45 to J44, J28 to J45, J29 to J46, J34 to J47, J35 to J48, J36 to J49, J53 to J5, J54 to J50, J37 to J51, J55 to J52, J38 to J53, J57 to J54, J14 to J6, J20 to J7, J44 to J8, J15 to J9, U1 to U8
Connections:
- net +BATT: now also P1.1; no longer P1.8
- net CURRENT: now also P1.3; no longer P1.6
- net GND: now also P1.2; no longer P1.7
- net M1: now also P1.5; no longer P1.4
- net M2: now also P1.6; no longer P1.3
- net M3: now also P1.7; no longer P1.2
- net M4: now also P1.8; no longer P1.1

Commit message: Add V0.3 known issues for V0.4 fix list, update open issues
C28 voltage rating, R30 divider, L2 inductor value, LED0 color,
LMR51430 upgrade path — all noted for next revision. CRIT-5 (ESC
connector) marked fixed. OSD pin mapping updated to GPIO4-6.

Co-Authored-By: Claude Opus 4.6 (1M context) <noreply@anthropic.com>
Parts:
- J16, J17, J19, J20, J23, J24, J3, J6, J9: now not fitted
Changed lines of the file:
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@@
 		(exclude_from_sim no)
 		(in_bom no)
-		(on_board yes)
+		(on_board no)
 		(in_pos_files yes)
-		(dnp no)
+		(dnp yes)
 		(property "Reference" "J16"
 			(at 77.216 25.654 90)
@@
 		(exclude_from_sim no)
 		(in_bom no)
-		(on_board yes)
+		(on_board no)
 		(in_pos_files yes)
-		(dnp no)
+		(dnp yes)
 		(property "Reference" "J19"
 			(at 83.566 25.654 90)
@@
 		(exclude_from_sim no)
 		(in_bom no)
-		(on_board yes)
+		(on_board no)
 		(in_pos_files yes)
-		(dnp no)
+		(dnp yes)
 		(property "Reference" "J23"
 			(at 89.916 25.654 90)
@@
 		(exclude_from_sim no)
 		(in_bom no)
-		(on_board yes)
+		(on_board no)
 		(in_pos_files yes)
-		(dnp no)
+		(dnp yes)
 		(property "Reference" "J17"
 			(at 77.216 54.864 90)
@@
 		(exclude_from_sim no)
 		(in_bom no)
-		(on_board yes)
+		(on_board no)
 		(in_pos_files yes)
-		(dnp no)
+		(dnp yes)
 		(property "Reference" "J9"
 			(at 56.896 25.654 90)
@@
 		(exclude_from_sim no)
 		(in_bom no)
-		(on_board yes)
+		(on_board no)
 		(in_pos_files yes)
-		(dnp no)
+		(dnp yes)
 		(property "Reference" "J6"
 			(at 50.546 25.654 90)
@@
 		(exclude_from_sim no)
 		(in_bom no)
-		(on_board yes)
+		(on_board no)
 		(in_pos_files yes)
-		(dnp no)
+		(dnp yes)
 		(property "Reference" "J20"
 			(at 83.566 54.864 90)
@@
 		(exclude_from_sim no)
 		(in_bom no)
-		(on_board yes)
+		(on_board no)
 		(in_pos_files yes)
-		(dnp no)
+		(dnp yes)
 		(property "Reference" "J3"
 			(at 44.196 25.654 90)
@@
 		(exclude_from_sim no)
 		(in_bom no)
-		(on_board yes)
+		(on_board no)
 		(in_pos_files yes)
-		(dnp no)
+		(dnp yes)
 		(property "Reference" "J24"
 			(at 89.916 54.864 90)
