File: hardware/power.kicad_sch (KiCad schematic)
At the start: 36 parts, among them Q1 DMN1150UFB-7B, U13 LP5912-3.3DRVR, U21 NCV8187AMT180TAG, U33 TPS2116DRLR, U6 LMR51420YFDDCR, U7 LMR51420YFDDCR

Commit message: WIP: schematic updates, library modernization, audit tooling
Schematic changes (user):
- Add ADC bypass caps on CURRENT/RSSI/EXTERNAL (1k + 100nF RC filter)
- Add IMU GYRO_CS 10k pull-up to +3.3V
- Reverse P1 ESC 8-pin JST SH pinout to BF standard
  (pin1=V+, pin2=GND, pin3=Current, pin5-8=M1-M4)
- SD card (blackbox) sub-sheet with SPI1 + FLASH_CS + decoupling
- Other sub-sheet cleanup (rp2350a, osd, pads, power, imu)

Footprint library:
- Convert all 62 legacy (module ...) footprints to modern
  (footprint ...) format via pcbnew API — fixes kicad-sch-api
  "footprint not found" errors

Tooling:
- Add hardware/tools/audit_design.py (BF-rule design audit script)
- Add hardware/tools/design_audit.md (audit report output)

Docs:
- Update CLAUDE.md: current GPIO map, corrected power tree net names,
  open issues list (CRIT-2..5), connector verification status

Co-Authored-By: Claude Opus 4.6 (1M context) <noreply@anthropic.com>
Parts:
- renumbered C35 to C24, C37 to C25, C36 to C26, C39 to C27, C38 to C28, C40 to C29, C48 to C30, C33 to C31, C2 to C33, C16 to C34, D5 to D4, D1 to D5, D21 to D6, D4 to D7, D7 to D8, L3 to L2, L4 to L3, Q1 to Q4, R7 to R27, R8 to R28, R14 to R29, R28 to R30, R16 to R31, R31 to R32, R29 to R33, R15 to R34, R19 to R35, R4 to R36, R12 to R37, U6 to U3, U7 to U4, U33 to U5, U21 to U6, U13 to U7

Commit message: V0.3 routed: pin remap, footprint fixes, EMC checklist, DFM prep
Schematic (user):
- OSD pins remapped to GPIO4-6 (OSD_W/OSD_EN/OSD_SYNC consecutive
  for FB_OSD PIO driver per BF PR#14882)
- SBUS inverter stays on GPIO9 (valid UART1_RX)
- Beeper moved to GPIO36
- Various sub-sheet updates

PCB:
- Full board routed, bottom-side component placement
- Resistor footprints: C_0201 -> R_0201 for correct 3D models
- Capacitor 3D model paths fixed (were pointing to R_0201)
- SD card footprint 3D path fixed (${KIPRJMOD}/lib.3dshapes/)
- 2 footprint 3D paths fixed (SIM, TF-01A: /lib.3dshapes -> ${KIPRJMOD})

Tooling & docs:
- Add EMC checklist (hardware/tools/EMC_CHECKLIST.md)
- Add EMC note script (hardware/tools/add_emc_note.py)
- Update CLAUDE.md: LMR51430 drop-in upgrade noted, connector
  verification, OSD pin mapping

Co-Authored-By: Claude Opus 4.6 (1M context) <noreply@anthropic.com>
Parts:
- removed D8: LED_1_Green, LED_SMD:LED_0201_0603Metric, symbol Device:LED
- removed R37: 200R, Capacitor_SMD:C_0201_0603Metric, symbol Device:R
- added D10: LED_1_Green, LED_SMD:LED_0201_0603Metric, symbol Device:LED
- added R40: 200R, Resistor_SMD:R_0201_0603Metric, symbol Device:R
- R27, R28, R29, R30, R31, R32, R33, R34, R35, R36: footprint Capacitor_SMD:C_0201_0603Metric -> Resistor_SMD:R_0201_0603Metric
Connections:
- net +5V: now also D10.2 (A)
- net at Q4.3 (D): now also R40.2
- new net: D10.1 (K), R40.1

Commit message: Add V0.3 known issues for V0.4 fix list, update open issues
C28 voltage rating, R30 divider, L2 inductor value, LED0 color,
LMR51430 upgrade path — all noted for next revision. CRIT-5 (ESC
connector) marked fixed. OSD pin mapping updated to GPIO4-6.

Co-Authored-By: Claude Opus 4.6 (1M context) <noreply@anthropic.com>
Parts:
- C30: value 22uF -> 4.7uF; footprint Capacitor_SMD:C_0603_1608Metric -> Capacitor_SMD:C_0402_1005Metric; LCSC C2762594 -> C23733; MPN CL10A226MO7JZNC -> CL05A475MP5NRNC
- L3: value XRTC303020D4R7MBCA -> FTC303020D100MBCA; LCSC Part C39846837 -> C7423323
Changed lines of the file:
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@@
 	)
 	(symbol
-		(lib_id "Device:C")
-		(at 146.05 160.02 0)
-		(unit 1)
-		(body_style 1)
-		(exclude_from_sim no)
-		(in_bom yes)
-		(on_board yes)
-		(in_pos_files yes)
-		(dnp no)
-		(fields_autoplaced yes)
-		(property "Reference" "C30"
-			(at 149.86 158.7499 0)
-			(show_name no)
-			(do_not_autoplace no)
-			(effects
-				(font
-					(size 1.27 1.27)
-				)
-				(justify left)
-			)
-		)
-		(property "Value" "22uF"
-			(at 149.86 161.2899 0)
-			(show_name no)
-			(do_not_autoplace no)
-			(effects
-				(font
-					(size 1.27 1.27)
-				)
-				(justify left)
-			)
-		)
-		(property "Footprint" "Capacitor_SMD:C_0603_1608Metric"
-			(at 147.0152 163.83 0)
-			(hide yes)
-			(show_name no)
-			(do_not_autoplace no)
-			(effects
-				(font
-					(size 1.27 1.27)
-				)
-			)
-		)
-		(property "Datasheet" ""
-			(at 146.05 160.02 0)
-			(hide yes)
-			(show_name no)
-			(do_not_autoplace no)
-			(effects
-				(font
-					(size 1.27 1.27)
-				)
-			)
-		)
-		(property "Description" "Unpolarized capacitor"
-			(at 146.05 160.02 0)
-			(hide yes)
-			(show_name no)
-			(do_not_autoplace no)
-			(effects
-				(font
-					(size 1.27 1.27)
-				)
-			)
-		)
-		(property "LCSC" "C2762594"
-			(at 146.05 160.02 0)
-			(hide yes)
-			(show_name no)
-			(do_not_autoplace no)
-			(effects
-				(font
-					(size 1.27 1.27)
-				)
-			)
-		)
-		(property "MPN" "CL10A226MO7JZNC"
-			(at 0 0 0)
-			(hide yes)
-			(show_name no)
-			(do_not_autoplace no)
-			(effects
-				(font
-					(size 1.27 1.27)
-				)
-			)
-		)
-		(property "Manufacturer" "Samsung Electro-Mechanics"
-			(at 0 0 0)
-			(hide yes)
-			(show_name no)
-			(do_not_autoplace no)
-			(effects
-				(font
-					(size 1.27 1.27)
-				)
-			)
-		)
-		(pin "1"
-		)
-		(pin "2"
-		)
-		(instances
-			(project "OpenFC"
-				(path "/fb88b6f9-ee39-4640-a9d4-04a17ceeac64/f8522f96-c979-41d2-ae00-e5ad899a3161"
-					(reference "C30")
-					(unit 1)
-				)
-			)
-		)
-	)
-	(symbol
 		(lib_id "Device:R")
 		(at 257.81 49.53 0)
@@
 			)
 		)
-		(property "Value" "XRTC303020D4R7MBCA"
+		(property "Value" "FTC303020D100MBCA"
 			(at 102.87 76.2 0)
 			(show_name no)
@@
 			)
 		)
-		(property "LCSC Part" "C39846837"
+		(property "LCSC Part" "C7423323"
 			(at 102.87 90.17 0)
 			(hide yes)
@@
 					(unit 1)
 				)
+			)
+		)
+	)
+	(symbol
+		(lib_id "Device:C")
+		(at 146.05 160.02 0)
+		(unit 1)
+		(body_style 1)
+		(exclude_from_sim no)
+		(in_bom yes)
+		(on_board yes)
+		(in_pos_files yes)
+		(dnp no)
+		(fields_autoplaced yes)
+		(property "Reference" "C30"
+			(at 149.86 158.7499 0)
+			(show_name no)
+			(do_not_autoplace no)
+			(effects
+				(font
+					(size 1.27 1.27)
+				)
+				(justify left)
+			)
+		)
+		(property "Value" "4.7uF"
+			(at 149.86 161.2899 0)
+			(show_name no)
+			(do_not_autoplace no)
+			(effects
+				(font
+					(size 1.27 1.27)
+				)
+				(justify left)
+			)
+		)
+		(property "Footprint" "Capacitor_SMD:C_0402_1005Metric"
+			(at 147.0152 163.83 0)
+			(hide yes)
+			(show_name no)
+			(do_not_autoplace no)
+			(effects
+				(font
+					(size 1.27 1.27)
+				)
+			)
+		)
+		(property "Datasheet" ""
+			(at 146.05 160.02 0)
+			(hide yes)
+			(show_name no)
+			(do_not_autoplace no)
+			(effects
+				(font
+					(size 1.27 1.27)
+				)
+			)
+		)
+		(property "Description" "Unpolarized capacitor"
+			(at 146.05 160.02 0)
+			(hide yes)
+			(show_name no)
+			(do_not_autoplace no)
+			(effects
+				(font
+					(size 1.27 1.27)
+				)
+			)
+		)
+		(property "LCSC" "C23733"
+			(at 146.05 160.02 0)
+			(hide yes)
+			(show_name no)
+			(do_not_autoplace no)
+			(effects
+				(font
+					(size 1.27 1.27)
+				)
+			)
+		)
+		(property "MPN" "CL05A475MP5NRNC"
+			(at -26.67 -41.91 0)
+			(hide yes)
+			(show_name no)
+			(do_not_autoplace no)
+			(effects
+				(font
+					(size 1.27 1.27)
+				)
+			)
+		)
+		(property "Manufacturer" "Samsung Electro-Mechanics"
+			(at -26.67 -41.91 0)
+			(hide yes)
+			(show_name no)
+			(do_not_autoplace no)
+			(effects
+				(font
+					(size 1.27 1.27)
+				)
+			)
+		)
+		(pin "1"
+		)
+		(pin "2"
+		)
+		(instances
+			(project "OpenFC"
+				(path "/fb88b6f9-ee39-4640-a9d4-04a17ceeac64/f8522f96-c979-41d2-ae00-e5ad899a3161"
+					(reference "C30")
+					(unit 1)
+				)

Commit message: Rev 2: fit 3A bucks, resolve power/LED/signal change-list items
Schematic (power, rp2350a) + docs in sync with Rev 2 decisions:

Power
- U3/U4 bucks: LMR51420 (2A) -> LMR51430YFDDCR (3A, C5219261)
- 10V FB R30 -> 6.49k (E96 stock) => Vout 9.85V
- C28 10V output cap kept 22uF 16V X5R 0603 (digital-VTX rail)
- L2/L3 both rails 4.7uH (XRTC303020D4R7MBCA)
- U6 gyro LDO kept NCV8187 (300mA) for PSRR

MCU/USB
- R12/R13/R14 kept at 30R (DFM consolidation, no impact)
- D1 USB ESD removed on schematic; flagged for restore (recommendation)

LEDs
- D2 LED0 -> blue XL-1005UBC; greens XL-1005UGC; all 0402
- Series resistors recalculated for ~1mA: D2 510R, D7 680R, D5 2.4k, D4 7.5k

Signals/decisions
- SBUS hardware inverter removed (BF PICO inverts at the RP2350 pad)
- Beeper done: N-MOS low-side (Q2 DMN1150UFB-7B)
- SDIO blackbox: stay on SPI (Betaflight PICO has no SDIO support)
- CRIT-2 motor order: keep reversed silk, fix in BF target resource map
- U5 confirmed TPS2116; SWD connector not added

Ignore generated analysis/ dump.

Co-Authored-By: Claude Opus 4.8 (1M context) <noreply@anthropic.com>
Parts:
- removed D10: LED_1_Green, LED_SMD:LED_0201_0603Metric, symbol Device:LED
- added D8: LED_1_Green, LED_SMD:LED_0402_1005Metric, symbol Device:LED
- D4, D5, D7: footprint LED_SMD:LED_0201_0603Metric -> LED_SMD:LED_0402_1005Metric; LCSC C3646922 -> C965793; MPN XL-0201UGC -> XL-1005UGC
- L3: value FTC303020D100MBCA -> XRTC303020D4R7MBCA; LCSC Part C7423323 -> C39846837
- R30: value 6.8k -> 6.49k; LCSC C274877 -> C474786
- U3, U4: value LMR51420YFDDCR -> TI LMR51430YFDDCR; LCSC Part C7296200 -> C5219261; MPN LMR51420YFDDCR -> TI LMR51430YFDDCR
Connections:
- net +5V: now also D8.2 (A)
- net at R40.1: now also D8.1 (K)
